File: Micro Tarea 2/Micro Tarea 2.kicad_pcb (KiCad board)
At the start: 4 copper layers, 70.8 x 86.7 mm, 62 parts, among them J1 Screw_Terminal_01x02, P1 USB_C_Plug_USB2.0, U7 TPS62130, U8 ESP32-S3R8, U9 W25Q128JVSIQ, Y1 40MHz

Commit message: actualizando placa
Parts:
- added SW1: K2-1157SP-I4SW-04, JLCImport:K2-1157SP-I4SW-04, F.Cu at (117.3, 101.5)
- added SW3: K2-1157SP-I4SW-04, JLCImport:K2-1157SP-I4SW-04, F.Cu at (117.3, 113.1)
- moved C29 66.7 mm to (115.7, 106.7), turned to 180 degrees
- moved D5 65.4 mm to (118.1, 94.1), turned to 180 degrees
- moved R2 57.4 mm to (119.3, 86.5)
- moved R3 54.9 mm to (119.3, 82.9)
- moved R34 54.7 mm to (119.2, 84.1)
- moved R35 54.4 mm to (119.2, 85.4)
- moved C39 50.6 mm to (132.1, 90.5), turned to -90 degrees
- moved C38 50.1 mm to (132.9, 88.5), turned to 180 degrees
- moved C40 49.7 mm to (130.9, 90.5), turned to -90 degrees
- moved C30 46.4 mm to (142.1, 99.5), turned to -90 degrees
- moved R21 46.2 mm to (118.7, 106.7), turned to 180 degrees
- moved C21 45.9 mm to (134.4, 114.3)
- moved C34 45.6 mm to (147.1, 95.3), turned to -90 degrees
- moved AE1 45.3 mm to (132.7, 81.3), turned to 90 degrees
- moved R23 45.1 mm to (135.0, 96.7), turned to 180 degrees
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Other:
- board size 70.8 x 86.7 mm -> 70.8 x 43.3 mm

Commit message: actualizando placa
Parts:
- moved TP6 9.07 mm to (124.0, 106.6)
Routing:
- net +3V3: track 0.00 -> 1.60 mm, vias 0 -> 13
- net GND: vias 0 -> 6
- added copper zone on F.Cu, net +3V3
- added copper zone on In2.Cu, net +3V3
- added copper zone on F.Cu, net GND
Changed lines of the file:
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@@
 	(footprint "TestPoint:TestPoint_Pad_D1.0mm"
 		(layer "F.Cu")
-		(at 129.02499 114.14688)
+		(at 124 106.6)
 		(descr "SMD pad as test Point, diameter 1.0mm")
 		(tags "test point SMD pad")
@@
 			(at 0 -1.448 0)
 			(layer "F.SilkS")
+			(hide yes)
 			(effects
 				(font
@@
 			(at 0 1.55 0)
 			(layer "F.Fab")
+			(hide yes)
 			(effects
 				(font
@@
 			(layer "F.CrtYd")
 		)
-		(fp_text user "${REFERENCE}"
-			(at 0 -1.45 0)
-			(layer "F.Fab")
-			(effects
-				(font
-					(size 1 1)
-					(thickness 0.15)
-				)
-			)
-		)
 		(pad "1" smd circle
 			(at 0 0)
@@
 		(layer "Edge.Cuts")
 	)
+	(segment
+		(start 124 106.6)
+		(end 125.6 106.6)
+		(width 0.4)
+		(layer "F.Cu")
+		(net "+3V3")
+	)
+	(via
+		(at 126.4 105.4)
+		(size 0.6)
+		(drill 0.3)
+		(layers "F.Cu" "B.Cu")
+		(free yes)
+		(net "+3V3")
+	)
+	(via
+		(at 128.8 105.4)
+		(size 0.6)
+		(drill 0.3)
+		(layers "F.Cu" "B.Cu")
+		(free yes)
+		(net "+3V3")
+	)
+	(via
+		(at 128 106.4)
+		(size 0.6)
+		(drill 0.3)
+		(layers "F.Cu" "B.Cu")
+		(free yes)
+		(net "+3V3")
+	)
+	(via
+		(at 126.4 106.4)
+		(size 0.6)
+		(drill 0.3)
+		(layers "F.Cu" "B.Cu")
+		(free yes)
+		(net "+3V3")
+	)
+	(via
+		(at 128.8 106.4)
+		(size 0.6)
+		(drill 0.3)
+		(layers "F.Cu" "B.Cu")
+		(free yes)
+		(net "+3V3")
+	)
+	(via
+		(at 128 105.4)
+		(size 0.6)
+		(drill 0.3)
+		(layers "F.Cu" "B.Cu")
+		(free yes)
+		(net "+3V3")
+	)
+	(via
+		(at 126.6 107.2)
+		(size 0.6)
+		(drill 0.3)
+		(layers "F.Cu" "B.Cu")
+		(free yes)
+		(net "+3V3")
+	)
+	(via
+		(at 130.4 106)
+		(size 0.6)
+		(drill 0.3)
+		(layers "F.Cu" "B.Cu")
+		(free yes)
+		(net "+3V3")
+	)
+	(via
+		(at 127.2 106.4)
+		(size 0.6)
+		(drill 0.3)
+		(layers "F.Cu" "B.Cu")
+		(free yes)
+		(net "+3V3")
+	)
+	(via
+		(at 129.6 106.4)
+		(size 0.6)
+		(drill 0.3)
+		(layers "F.Cu" "B.Cu")
+		(free yes)
+		(net "+3V3")
+	)
+	(via
+		(at 129.6 105.4)
+		(size 0.6)
+		(drill 0.3)
+		(layers "F.Cu" "B.Cu")
+		(free yes)
+		(net "+3V3")
+	)
+	(via
+		(at 127.2 105.4)
+		(size 0.6)
+		(drill 0.3)
+		(layers "F.Cu" "B.Cu")
+		(free yes)
+		(net "+3V3")
+	)
+	(via
+		(at 129 107.2)
+		(size 0.6)
+		(drill 0.3)
+		(layers "F.Cu" "B.Cu")
+		(free yes)
+		(net "+3V3")
+	)
+	(via
+		(at 130 111.8)
+		(size 0.6)
+		(drill 0.3)
+		(layers "F.Cu" "B.Cu")
+		(free yes)
+		(net "GND")
+	)
+	(via
+		(at 128.4 111.8)
+		(size 0.6)
+		(drill 0.3)
+		(layers "F.Cu" "B.Cu")
+		(free yes)
+		(net "GND")
+	)
+	(via
+		(at 129.2 111.8)
+		(size 0.6)
+		(drill 0.3)
+		(layers "F.Cu" "B.Cu")
+		(free yes)
+		(net "GND")
+	)
+	(via
+		(at 126.8 111.8)
+		(size 0.6)
+		(drill 0.3)
+		(layers "F.Cu" "B.Cu")
+		(free yes)
+		(net "GND")
+	)
+	(via
+		(at 126 111.8)
+		(size 0.6)
+		(drill 0.3)
+		(layers "F.Cu" "B.Cu")
+		(free yes)
+		(net "GND")
+	)
+	(via
+		(at 127.6 111.8)
+		(size 0.6)
+		(drill 0.3)
+		(layers "F.Cu" "B.Cu")
+		(free yes)
+		(net "GND")
+	)
+	(zone
+		(net "+3V3")
+		(layer "F.Cu")
+		(hatch edge 0.5)
+		(priority 2)
+		(connect_pads
+			(clearance 0.5)
+		)
+		(min_thickness 0.25)
+		(fill yes
+			(thermal_gap 0.5)
+			(thermal_bridge_width 0.5)
+			(island_removal_mode 0)
+		)
+		(polygon
+			(pts
+				(xy 133.6 104.6) (xy 133.62499 109.6) (xy 134.4 110.4) (xy 134.42499 111.2) (xy 131.6 111.2) (xy 130.4 109.4)
+				(xy 125.4 109.4) (xy 125.4 104.6)
+			)
+		)
+	)
+	(zone
+		(net "GND")
+		(locked yes)
+		(layer "F.Cu")
+		(hatch edge 0.5)
+		(priority 3)
+		(connect_pads
+			(clearance 0.5)
+		)
+		(min_thickness 0.25)
+		(fill yes
+			(thermal_gap 0.5)
+			(thermal_bridge_width 0.5)
+			(island_removal_mode 0)
+		)
+		(polygon
+			(pts
+				(xy 125.6 109.6) (xy 129.8 109.54688) (xy 130.6 110.8) (xy 130.6 112.6) (xy 125.2 112.6) (xy 125.2 109.6)
+			)
+		)
+	)
 	(zone
 		(net "GND")
+		(locked yes)
 		(layer "In1.Cu")
 		(hatch edge 0.5)
@@
 			)
 		)
+	)
+	(zone
+		(net "+3V3")
+		(locked yes)
+		(layer "In2.Cu")
+		(hatch edge 0.5)
+		(priority 1)
+		(connect_pads
+			(clearance 0.5)
+		)
+		(min_thickness 0.25)
+		(fill yes
+			(thermal_gap 0.5)
+			(thermal_bridge_width 0.5)
+			(island_removal_mode 0)
+		)
+		(polygon
+			(pts
+				(xy 110.6 77) (xy 181 76.8) (xy 181 119.8) (xy 110.6 119.8)
+			)
+		)
